File: AD Envelope.kicad_sch (KiCad schematic)
At the start: 92 parts, among them J1 Conn_02x05_Odd_Even, J10 Conn_01x01, J11 Conn_01x01, J12 Conn_01x01, J13 Conn_01x01, J14 Conn_01x01, J15 Conn_01x01, J16 Conn_01x01, J17 Conn_01x01, J2 Conn_01x01, J3 Conn_01x01, J4 Conn_01x01, J5 Conn_01x01, J6 Conn_01x01, J7 Conn_01x01, J8 Conn_01x01, J9 Conn_01x01, Q1 BC556, Q2 BC556, Q3 BC556, Q4 BC546, SW1 SW_SPDT, SW2 SW_SPDT, SW3 SW_SPDT_MSM, SW4 SW_SPST, U1 TL072, U2 TL072, U3 4011, U4 4013

Commit message: exponential version wip
Parts:
- removed C1: 10u, Capacitor_THT:CP_Radial_D6.3mm_P2.50mm, symbol Device:C_Polarized
- removed C14: 0.1n, Capacitor_THT:C_Disc_D5.1mm_W3.2mm_P5.00mm, symbol Device:C
- removed C2: 1u, Capacitor_THT:C_Rect_L7.2mm_W5.0mm_P5.00mm, symbol Device:C
- removed D3, D7: 1N4148, Diode_THT:D_DO-35_SOD27_P7.62mm_Horizontal, symbol Diode:1N4148
- removed J6, J7, J8: Conn_01x01, Connector_Pin:Pin_D1.0mm_L10.0mm, symbol Connector_Generic:Conn_01x01
- removed JP1, JP2, JP3, JP5: Jumper_2_Bridged, Jumpers:Jumper_P6.00mm, symbol Jumper:Jumper_2_Bridged
- removed JP10, JP11, JP6, JP8: Jumper_2_Bridged, Jumpers:Jumper_P8.00mm, symbol Jumper:Jumper_2_Bridged
- removed JP4: Jumper_2_Bridged, Jumpers:Jumper_P14.00mm, symbol Jumper:Jumper_2_Bridged
- removed JP7: Jumper_2_Bridged, Jumpers:Jumper_P18.00mm, symbol Jumper:Jumper_2_Bridged
- removed JP9: Jumper_2_Bridged, Jumpers:Jumper_P10.00mm, symbol Jumper:Jumper_2_Bridged
- removed Q1, Q3: BC556, Package_TO_SOT_THT:TO-92_Wide, symbol Transistor_BJT:BC556
- removed R13, R19: 22k, Resistor_THT:R_Axial_DIN0207_L6.3mm_D2.5mm_P10.16mm_Horizontal, symbol Device:R
- removed R15: 100k, Resistor_THT:R_Axial_DIN0207_L6.3mm_D2.5mm_P10.16mm_Horizontal, symbol Device:R
- removed R22: 10k, Resistor_THT:R_Axial_DIN0207_L6.3mm_D2.5mm_P10.16mm_Horizontal, symbol Device:R
- removed R6: 1k, Resistor_THT:R_Axial_DIN0207_L6.3mm_D2.5mm_P10.16mm_Horizontal, symbol Device:R
- removed RV1: 1M, symbol Device:R_Potentiometer
- removed SW1, SW2: SW_SPDT, Button_Switch_SMD:Nidec_Copal_CAS-120A, symbol Switch:SW_SPDT
- removed SW3: SW_SPDT_MSM, Button_Switch_SMD:Nidec_Copal_CAS-120A, symbol Switch:SW_SPDT_MSM
- added C1, C13: 0.1n, Capacitor_THT:C_Disc_D5.1mm_W3.2mm_P5.00mm, symbol Device:C
- added C12, C16, C17: 0.1u, Capacitor_THT:C_Disc_D5.1mm_W3.2mm_P5.00mm, symbol Device:C
- added C3: 10n, Capacitor_THT:C_Disc_D5.1mm_W3.2mm_P5.00mm, symbol Device:C
- added D4: 1N4148, Diode_THT:D_DO-35_SOD27_P7.62mm_Horizontal, symbol Diode:1N4148
- added Q1, Q2: AS394CH, Package_TO_SOT_THT:TO-5-8, symbol Transistors:AS394CH
- added Q10, Q6, Q9: BS170, Package_TO_SOT_THT:TO-92_Wide, symbol Transistor_FET:BS170
- added Q3: AS395H, Package_TO_SOT_THT:TO-5-8, symbol Transistors:AS395H
- added Q5: BC556, Package_TO_SOT_THT:TO-92_Wide, symbol Transistor_BJT:BC556
- added Q7: BC546, Package_TO_SOT_THT:TO-92_Wide, symbol Transistor_BJT:BC546
- added R18: 22k, Resistor_THT:R_Axial_DIN0207_L6.3mm_D2.5mm_P10.16mm_Horizontal, symbol Device:R
- added R8: 1k, Resistor_THT:R_Axial_DIN0207_L6.3mm_D2.5mm_P10.16mm_Horizontal, symbol Device:R
- added RV1, RV3: 50k, Potentiometer_THT:Potentiometer_Bourns_3296Y_Vertical, symbol Device:R_Potentiometer_Trim
- added RV4: 1k, Package_SO:TSSOP-20_4.4x6.5mm_P0.65mm, symbol Device:R_Potentiometer
- added U1: 40106, Package_DIP:DIP-14_W7.62mm_Socket, symbol 4xxx:40106
- added U5: DG419LDJ, Package_DIP:DIP-8_W7.62mm_Socket, symbol Analog_Switch:DG419LDJ
- added U6: LM311, Package_DIP:DIP-8_W7.62mm_Socket, symbol Comparator:LM311
- C2: renamed from C3; footprint Capacitor_THT:C_Rect_L7.2mm_W2.5mm_P5.00mm -> Capacitor_THT:C_Rect_L10.3mm_W4.5mm_P7.50mm_MKS4
- R1: value 9.1k -> 1.2k 1%
- R10: value 22k -> 100k
- R11: value 1k -> 100
- R14, R16: value 100k -> 10k
- R17, R20: value 22k -> 10k
- R2, R5: value 1k -> 1M
- R3: value 1k -> 10k
- R4: value 9.1k -> 470
- R7: value 22k -> 100
- R9: value 10k -> 22k
- RV2: value 1M -> 1k; footprint (none) -> Package_SO:TSSOP-20_4.4x6.5mm_P0.65mm
- renumbered C9 to C10, C5 to C11, C10 to C14, C11 to C15, C6 to C5, C7 to C6, C12 to C7, C13 to C8, C8 to C9, D4 to D3, J13 to J10, J14 to J11, J15 to J12, J16 to J13, J17 to J14, J9 to J6, J10 to J7, J11 to J8, J12 to J9, Q2 to Q8, R18 to R13, R21 to R15, R24 to R19, R25 to R21, R23 to R22, R8 to R6, SW4 to SW1, U4 to U2, U2 to U3, U1 to U4, U3 to U7
Connections:
- net VCC2 is gone; now on net VCC: C14.1, C9.1, U3.8 (V+), U4.8 (V+)
- net CLK: now also U2.11 (C), U7.5, U7.6, R18.1, U1.4, U5.6; no longer U2.3 (C), U7.2
- net CYCLE_EN: now also D4.2 (A); no longer R15.2
- net GND: now also D2.1 (K), D6.2 (A), R10.1, RV2.1, U2.3 (C), U2.4 (R), U2.5 (D), U2.6 (S), U4.5 (+), C12.2, C13.2, C16.2, C17.1, Q1.6 (B2), Q10.3 (S), Q2.6 (B2), RV4.1, U1.11, U1.5, U1.7 (VSS), U5.3 (GND), U6.1 (GND); no longer U2.10 (R), U2.11 (C), U2.8 (S), U2.9 (D), U3.3 (+), U7.12, U7.13
- net RAMP_OUT: now also R8.1; no longer R11.1
- net TRIG_IN: now also R17.2
- net VCC: now also C11.1, C7.1, C8.1, D5.1 (K), R1.2, R14.2, R16.2, R3.2, U2.14 (VDD), U2.9 (D), U7.14 (VDD), C12.1, C16.1, C3.1, Q3.3 (E1), Q3.5 (E2), Q7.1 (C), RV1.1, RV1.2, RV3.1, RV3.2, U1.14 (VDD), U5.4 (V+), U5.5 (VL), U6.8 (V+)
- net VEE: now also C10.2, C15.2, R13.2, U3.4 (V-), U4.4 (V-), C17.2, Q9.3 (S), U5.7 (V-), U6.4 (V-)
- net at Q4.1 (C): now also Q3.1 (C1), Q5.2 (B)
- net at Q4.3 (E): now also Q1.7 (C2)
- net at C11.2, R20.1: now also U2.8 (S); no longer U2.6 (S)
- net R_CV: now reaches U3.6 (-)
- net R_CV: now also U3.7, Q2.2 (B1)
- net at R9.2: now also Q9.1 (D), U6.3 (-)
- net ~{Q}: now reaches U2.12 (~{Q})
- net ~{Q}: now also U7.1
- net Q: now reaches U2.13 (Q)
- net Q: now also R7.2
- net at C4.2, R15.1: now also U1.8; no longer U4.6 (-), U4.7
- net at R3.1: now also D1.2 (A), Q4.2 (B)
- net at C4.1, R13.1: now also R11.2; no longer R16.2
- net at U7.3: now also U7.12, U7.13
- net at U7.8, U7.9: now also U1.12
- net at R12.1: now also R10.2, U6.2 (+); no longer R9.1
- net at R17.1: now also D5.2 (A), D6.1 (K), Q10.2 (G); no longer U3.5 (+)
- net at R21.1: now also U7.11; no longer U7.10
- net CMP_OUT: now reaches R14.1
- net CMP_OUT: now also R12.2, U1.1, U6.7
- net FALL_OUT renamed F_OUT
- removed net F_FAST: D2.2 (A), J4.1 (Pin_1), R4.1
- removed net F_SLOW: J5.1 (Pin_1), R4.2, R5.2
- removed net INT_IN: C2.1, RV2.2, RV2.3, U4.2 (-)
- net RISE_OUT renamed R_OUT
- removed net R_FAST: D1.1 (K), J2.1 (Pin_1), R1.1
- removed net R_SLOW: J3.1 (Pin_1), R1.2, R2.2
- removed net ST_OUT: D1.2 (A), D2.1 (K), D6.2 (A), U3.7
- removed net VCC1: C11.1, C7.1, C8.1, U2.14 (VDD), U2.5 (D), U7.14 (VDD)
- removed net VEE1: C10.2, C15.2, D5.2 (A), R12.2, R13.2, U3.4 (V-), U4.4 (V-)
- new net: Q9.2 (G), R11.1
- new net: C1.1, Q1.1 (C1), Q2.1 (C1), R1.1, U4.2 (-)
- new net: D1.1 (K), D2.2 (A)
- new net: Q1.3 (E1), Q1.5 (E2), R2.2, U5.2
- new net: C1.2, R4.1, U4.1
- new net: R4.2, U5.1
- new net: C2.1, Q2.7 (C2), Q5.1 (C), Q6.3 (S), U4.6 (-)
- new net: Q3.2 (B1), Q3.6 (B2), Q3.7 (C2), Q5.3 (E)
- new net: Q2.3 (E1), Q2.5 (E2), R5.2, U5.8
- new net: Q10.1 (D), R16.1, U1.9
- new net: C13.1, R18.2, U1.13
- new net: Q7.3 (E), R6.1
- new net: Q6.2 (G), R7.1
- new net: U7.10, U7.2
- new net: U1.2, U1.3
- new net: C3.2, U6.5 (BAL), U6.6 (STRB)
- new net F_CV: Q1.2 (B1), U3.1, U3.2 (-)
- new net F_POT_IN: J4.1 (Pin_1), RV3.3, RV4.3
- new net F_POT_WIPER: J5.1 (Pin_1), RV4.2, U3.3 (+)
- new net INT_OUT: C2.2, Q6.1 (D), Q7.2 (B), R8.2, R9.1, U4.7
- new net RESET: D4.1 (K), R15.2, U2.10 (R)
- new net R_POT_IN: J2.1 (Pin_1), RV1.3, RV2.3
- new net R_POT_WIPER: J3.1 (Pin_1), RV2.2, U3.5 (+)
Other:
- note removed: "Front panel"
- moved on the sheet: C10, C11, C14, C15, C2, C4, C5, C6, C7, C8, C9, D3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

Commit message: delete jumpers library
Parts:
- removed RV3: 50k, Potentiometer_THT:Potentiometer_Bourns_3296Y_Vertical, symbol Device:R_Potentiometer_Trim
- removed U3: TL072, Package_DIP:DIP-8_W7.62mm_Socket, symbol Amplifier_Operational:TL072
- added C16, C17, C18, C19: 0.1u, Capacitor_THT:C_Disc_D5.1mm_W3.2mm_P5.00mm, symbol Device:C
- added J10, J6, J7, J8, J9: Conn_01x01, Connector_Pin:Pin_D1.0mm_L10.0mm, symbol Connector_Generic:Conn_01x01
- added R1, R2: 33k, Resistor_THT:R_Axial_DIN0207_L6.3mm_D2.5mm_P10.16mm_Horizontal, symbol Device:R
- added R10, R11, R12, R3, R4, R5, R6, R7, R8, R9: 22k, Resistor_THT:R_Axial_DIN0207_L6.3mm_D2.5mm_P10.16mm_Horizontal, symbol Device:R
- added RV1, RV6: 1k, Package_SO:TSSOP-20_4.4x6.5mm_P0.65mm, symbol Device:R_Potentiometer
- added RV5: 50k, Potentiometer_THT:Potentiometer_Bourns_3296Y_Vertical, symbol Device:R_Potentiometer_Trim
- added SW1: SW_SPDT, Package_SON:WSON-8-1EP_6x5mm_P1.27mm_EP3.4x4mm, symbol Switch:SW_SPDT
- added U3, U4: TL074, Package_DIP:DIP-14_W7.62mm_Socket, symbol Amplifier_Operational:TL074
- R24: renamed from R12; value 10k -> 22k
- R26: renamed from R14; value 10k -> 2.2k
- renumbered C12 to C11, C14 to C12, C15 to C13, C16 to C14, C17 to C15, C11 to C20, C13 to C21, C5 to C3, C6 to C4, C7 to C5, C3 to C6, C8 to C7, C4 to C8, J6 to J11, J7 to J12, J8 to J13, J9 to J14, J10 to J15, J11 to J16, J12 to J17, J13 to J18, J14 to J19, R1 to R13, R2 to R14, R3 to R15, R4 to R16, R5 to R17, R6 to R18, R7 to R19, R8 to R20, R9 to R21, R10 to R22, R11 to R23, R13 to R25, R15 to R27, R16 to R28, R17 to R29, R18 to R30, R19 to R31, R20 to R32, R21 to R33, R22 to R34, RV1 to RV2, RV2 to RV3, SW1 to SW2, U4 to U5, U5 to U6, U6 to U7, U7 to U8
Connections:
- net CLK: now also U1.8, U2.3 (C); no longer U1.4, U2.11 (C)
- net CMP_OUT: now also U1.11; no longer U1.1
- net F_CV: now also R12.1, U4.7
- net F_POT_IN: now also RV5.3, RV6.3; no longer RV4.3
- net GND: now also U1.13, U2.10 (R), U2.11 (C), U2.8 (S), U2.9 (D), C16.2, C17.1, C18.2, C19.1, RV1.1, RV6.1, U3.3 (+), U3.5 (+), U4.3 (+), U4.5 (+); no longer U1.11, U2.3 (C), U2.4 (R), U2.5 (D), U2.6 (S)
- net Q: now also U2.1 (Q); no longer U2.13 (Q)
- net RESET: now also U2.4 (R); no longer U2.10 (R)
- net R_CV: now also R11.1, U3.7
- net VCC: now also U2.5 (D), C16.1, C18.1, RV5.1, RV5.2, U3.4 (V+), U4.4 (V+); no longer U2.9 (D)
- net VEE: now also C17.2, C19.2, U3.11 (V-), U4.11 (V-)
- net ~{Q}: now also U2.2 (~{Q}); no longer U2.12 (~{Q})
- net at C20.2, R32.1: now also U2.6 (S); no longer U2.8 (S)
- net at C8.2, R27.1: now also U1.2; no longer U1.8
- net at Q10.1 (D), R28.1: now also U1.1; no longer U1.9
- net at C21.1, R30.2: now also U1.3; no longer U1.13
- net at U8.8, U8.9: now also U1.4; no longer U1.12
- net at U1.10: now also U1.9
- net F_POT_WIPER renamed F_CV_WIPER
- net F_CV_WIPER: now also J7.1 (Pin_1), U4.10 (+); no longer J5.1 (Pin_1)
- net R_POT_WIPER renamed R_WIPER
- net R_WIPER: now also U3.12 (+)
- new net: R1.1, RV1.3
- new net: R3.1, R6.1, R8.2, U4.2 (-)
- new net: R3.2, U4.13 (-), U4.14
- new net: R7.1, R9.2, U3.1
- new net: R4.1, R5.1, R7.2, U3.2 (-)
- new net: R5.2, U3.13 (-), U3.14
- new net: R2.1, RV4.3
- new net: R10.1, R12.2, U4.6 (-)
- new net: R11.2, R9.1, U3.6 (-)
- new net: R10.2, R8.1, U4.1
- new net F_CV_BUF: J9.1 (Pin_1), SW1.1 (A), U4.8, U4.9 (-)
- new net F_CV_IN: R2.2
- new net F_CV_SUM_IN: J10.1 (Pin_1), R6.2, SW1.2 (B)
- new net F_WIPER: J5.1 (Pin_1), RV6.2, U4.12 (+)
- new net R_CV_BUF: J8.1 (Pin_1), R4.2, SW1.3 (C), U3.8, U3.9 (-)
- new net R_CV_IN: R1.2
- new net R_CV_WIPER: J6.1 (Pin_1), RV1.2, U3.10 (+)
Other:
- note added: "Front panel"
- title: (none) -> Ramp generator
- moved on the sheet: C1, C2, C20, C21, C6, C8, D1, D2, D3, D4, D5, D6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

Commit message: small tweaks
Parts:
- removed C16, C17, C19: 0.1u, Capacitor_THT:C_Disc_D5.1mm_W3.2mm_P5.00mm, symbol Device:C
- removed C6: 10n, Capacitor_THT:C_Disc_D5.1mm_W3.2mm_P5.00mm, symbol Device:C
- removed Q1: AS394CH, Package_TO_SOT_THT:TO-5-8, symbol Transistors:AS394CH
- removed Q5: BC556, Package_TO_SOT_THT:TO-92_Wide, symbol Transistor_BJT:BC556
- removed Q7: BC546, Package_TO_SOT_THT:TO-92_Wide, symbol Transistor_BJT:BC546
- removed R10: 22k, Resistor_THT:R_Axial_DIN0207_L6.3mm_D2.5mm_P10.16mm_Horizontal, symbol Device:R
- removed R17: 1M, Resistor_THT:R_Axial_DIN0207_L6.3mm_D2.5mm_P10.16mm_Horizontal, symbol Device:R
- removed unit 4 of U1
- removed unit 5 of U1
- removed U5: TL072, Package_DIP:DIP-8_W7.62mm_Socket, symbol Amplifier_Operational:TL072
- removed U6: DG419LDJ, Package_DIP:DIP-8_W7.62mm_Socket, symbol Analog_Switch:DG419LDJ
- removed U7: LM311, Package_DIP:DIP-8_W7.62mm_Socket, symbol Comparator:LM311
- added C2: 0.1n, Capacitor_THT:C_Disc_D5.1mm_W3.2mm_P5.00mm, symbol Device:C
- added D4, D5: 1N4148, Diode_THT:D_DO-35_SOD27_P7.62mm_Horizontal, symbol Diode:1N4148
- added J1, J2, J22, J23, J24: CV, symbol Connector_Audio:AudioJack2
- added R11: 2.2M, Resistor_THT:R_Axial_DIN0207_L6.3mm_D2.5mm_P10.16mm_Horizontal, symbol Device:R
- added R27: 10k, Resistor_THT:R_Axial_DIN0207_L6.3mm_D2.5mm_P10.16mm_Horizontal, symbol Device:R
- added R29: 47k, Resistor_THT:R_Axial_DIN0207_L6.3mm_D2.5mm_P10.16mm_Horizontal, symbol Device:R
- added U3: TL074, Package_DIP:DIP-14_W7.62mm_Socket, symbol Amplifier_Operational:TL074
- added unit 2 of U6
- added unit 5 of U6
- C18: value 0.1u -> 1n
- C3: renamed from C2; value 0.1u -> 47n; footprint Capacitor_THT:C_Rect_L10.3mm_W4.5mm_P7.50mm_MKS4 -> Capacitor_THT:C_Rect_L13.0mm_W5.0mm_P10.00mm_FKS3_FKP3_MKS4
- R10: renamed from R11; value 22k -> 10k
- R12: value 22k -> 2.2M
- R13: value 1.2k 1% -> 2.2k 1%
- R14: value 1M -> 2.2k 1%
- R15: value 10k -> 820
- R16: value 470 -> 820
- R20: renamed from R21; value 22k -> 10k
- R21: renamed from R22; value 100k -> 68k
- R23: renamed from R24; value 22k -> 10k
- R25: renamed from R27; value 22k -> 33k
- R26: value 2.2k -> 10k
- R3: renamed from R5; value 22k -> 10k
- R4: renamed from R3; value 22k -> 10k
- R5: renamed from R4; value 22k -> 10k
- R6, R9: value 22k -> 10k
- R7: renamed from R8; value 22k -> 10k
- R8: renamed from R7; value 22k -> 10k
- renumbered C11 to C10, C12 to C11, C13 to C12, C14 to C13, C15 to C14, C8 to C15, C20 to C16, C21 to C17, C3 to C4, C4 to C5, C5 to C6, C9 to C8, C10 to C9, D4 to D6, D5 to D7, D6 to D8, J8 to J10, J9 to J11, J10 to J12, J11 to J13, J12 to J14, J13 to J15, J14 to J16, J15 to J17, J16 to J18, J17 to J19, J18 to J20, J19 to J21, J1 to J3, J2 to J4, J3 to J5, J4 to J6, J5 to J7, J6 to J8, J7 to J9, Q3 to Q1, Q6 to Q3, Q8 to Q5, Q9 to Q6, Q10 to Q7, R2 to R1, R20 to R17, R19 to R18, R18 to R19, R1 to R2, R23 to R22, R25 to R24, R30 to R28, R32 to R30, R28 to R31, R29 to R32, R31 to R33, R33 to R34, R34 to R35, RV4 to RV1, RV6 to RV2, RV1 to RV3, RV3 to RV4, RV2 to RV5, RV5 to RV6, U4 to U1, U3 to U2, U2 to U4, U8 to U5, U1 to U6
Connections:
- net CLK: now also R26.2, U5.12, U5.13, D5.1 (K); no longer U5.5, U5.6
- net CMP_OUT: now also D1.1 (K), D2.2 (A), D4.2 (A), U3.1; no longer R23.2
- net F_CV: now also Q1.6 (B2), R7.1, U1.7; no longer R12.1, U1.7
- net F_CV_BUF: now also U1.13 (-), U1.14; no longer U1.8, U1.9 (-)
- net F_CV_IN: now also J2.T
- net F_CV_WIPER: now also U1.12 (+); no longer U1.10 (+)
- net F_OUT: now also J24.T
- net F_WIPER: now also U1.10 (+); no longer U1.12 (+)
- net GND: now also Q1.2 (B1), U1.3 (+), U1.5 (+), U2.3 (+), U6.1, D5.2 (A), J1.S, J2.S, J22.S, J23.S, J24.S, U3.10 (+), U3.12 (+), U3.5 (+), U6.11, U6.3; no longer C18.2, D2.1 (K), R14.1, U1.3 (+), U1.5 (+), U2.3 (+), U6.13
- net INT_OUT: now also Q4.2 (B), U3.7
- net RAMP_OUT: now also J22.T
- net R_CV: now also U1.1; no longer U2.7
- net R_CV_BUF: now also U2.13 (-), U2.14; no longer U2.8, U2.9 (-)
- net R_CV_IN: now also J1.T
- net R_CV_WIPER: now also U2.12 (+); no longer U2.10 (+)
- net R_OUT: now also J23.T
- net R_WIPER: now also U2.10 (+); no longer U2.12 (+)
- net VCC: now also Q4.1 (C), R12.1, R29.2, U3.4 (V+); no longer C18.1, Q1.3 (E1), Q1.5 (E2), R13.2, R15.2, R26.2
- net VEE: now also R11.1, U3.11 (V-)
- net at R4.1, R6.1, R7.2: now also U1.6 (-); no longer U1.2 (-)
- net at C1.1, Q2.1 (C1): now also R14.1, U3.13 (-); no longer R13.1
- net at R14.2: now also D2.1 (K), R12.2
- net at C1.2, R16.1: now also U3.14
- net at R16.2: now also Q2.3 (E1), Q2.5 (E2)
- net at R8.1, R9.2: now also U2.7; no longer U2.1
- net at R3.1, R5.1, R8.2: now also U2.6 (-); no longer U2.2 (-)
- net at C3.1, Q2.7 (C2), Q3.3 (S): now also Q1.1 (C1), U3.6 (-)
- net at R23.1: now also D4.1 (K); no longer R21.2
- net at C15.2, R25.1: now also U6.12; no longer U6.2
- net at Q7.1 (D), R31.1: now also C18.2; no longer U6.1
- net at C17.1, R28.2: now also U6.9; no longer U6.3
- net at R35.1: now also U5.11; no longer U5.4
- net at R19.1: now also Q4.3 (E)
- net at R34.1: now also U5.10; no longer U5.11
- net at U5.2: now also U5.4; no longer U5.10
- net at R10.2, R9.1: now also U1.2 (-); no longer U2.6 (-)
- net at Q6.1 (D), R20.2: now also U3.2 (-)
- new net: C18.1, R27.1, R29.1
- new net: D1.2 (A), R11.2, R13.1
- new net: C2.1, Q1.7 (C2), R13.2, U3.9 (-)
- new net: C2.2, R15.2, U3.8
- new net: R21.2, R23.2, U3.3 (+)
- new net: Q1.3 (E1), Q1.5 (E2), R15.1
- new net: U2.1, U2.2 (-)
- new net: R3.2, U2.8, U2.9 (-)
- new net: U5.3, U5.8, U5.9
- new net: R4.2, U1.8, U1.9 (-)
- new net: U5.5, U5.6, U6.8
- new net: R27.2, U6.13
Other:
- moved on the sheet: C1, C10, C11, C12, C13, C14, C15, C16, C17, C3, C4, C5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

Commit message: threshold pot
Parts:
- removed R21: 68k, Resistor_THT:R_Axial_DIN0207_L6.3mm_D2.5mm_P10.16mm_Horizontal, symbol Device:R
- added RV7: 50k, Potentiometer_THT:Potentiometer_Bourns_3296Y_Vertical, symbol Device:R_Potentiometer_Trim
- renumbered R22 to R21, R24 to R22, R25 to R24, R26 to R25, R27 to R26, R28 to R27, R29 to R28, R30 to R29, R31 to R30, R32 to R31, R33 to R32, R34 to R33, R35 to R34
Connections:
- net GND: now also R23.2
- net at D4.1 (K): now also RV7.3; no longer R23.1
- net at U3.3 (+): now also RV7.2; no longer R23.2
- new net: R23.1, RV7.1
Other:
- note added: "Threshold / peak trim"
- moved on the sheet: R23
