File: AD Envelope.kicad_pcb (KiCad board)
At the start: 2 copper layers, 75 x 100 mm, 83 parts, among them J1 Conn_02x05_Odd_Even, J10 Conn_01x01, J11 Conn_01x01, J12 Conn_01x01, J13 Conn_01x01, J14 Conn_01x01, J15 Conn_01x01, J16 Conn_01x01, J17 Conn_01x01, J2 Conn_01x01, J3 Conn_01x01, J4 Conn_01x01, J5 Conn_01x01, J6 Conn_01x01, J7 Conn_01x01, J8 Conn_01x01, J9 Conn_01x01, Q1 BC556, Q2 BC556, Q3 BC556, Q4 BC546, U1 TL072, U2 TL072, U3 4011, U4 4013

Commit message: exponential version wip
Parts:
- removed D3, D7: 1N4148, Diode_THT:D_DO-35_SOD27_P7.62mm_Horizontal
- removed J15, J16, J17: Conn_01x01, Connector_Pin:Pin_D1.0mm_L10.0mm
- removed JP1, JP2, JP3, JP5: Jumper_2_Bridged, Jumpers:Jumper_P6.00mm
- removed JP10, JP11, JP6, JP8: Jumper_2_Bridged, Jumpers:Jumper_P8.00mm
- removed JP4: Jumper_2_Bridged, Jumpers:Jumper_P14.00mm
- removed JP7: Jumper_2_Bridged, Jumpers:Jumper_P18.00mm
- removed JP9: Jumper_2_Bridged, Jumpers:Jumper_P10.00mm
- removed R23, R25: 1k, Resistor_THT:R_Axial_DIN0207_L6.3mm_D2.5mm_P10.16mm_Horizontal
- removed R24: 100k, Resistor_THT:R_Axial_DIN0207_L6.3mm_D2.5mm_P10.16mm_Horizontal
- added C15: 0.1u, Capacitor_THT:C_Disc_D5.1mm_W3.2mm_P5.00mm, F.Cu at (46.2, 38.4)
- added C16: 0.1u, Capacitor_THT:C_Disc_D5.1mm_W3.2mm_P5.00mm, F.Cu at (54.3, 28.9)
- added C17: 0.1u, Capacitor_THT:C_Disc_D5.1mm_W3.2mm_P5.00mm, F.Cu at (54.3, 33.6)
- added D4: 1N4148, Diode_THT:D_DO-35_SOD27_P7.62mm_Horizontal, F.Cu at (173.5, 104.3)
- added Q10: BS170, Package_TO_SOT_THT:TO-92_Wide, F.Cu at (214.7, 97.7)
- added Q5: BC556, Package_TO_SOT_THT:TO-92_Wide, F.Cu at (141.8, 64.0)
- added Q6: BS170, Package_TO_SOT_THT:TO-92_Wide, F.Cu at (149.2, 126.0)
- added Q7: BC546, Package_TO_SOT_THT:TO-92_Wide, F.Cu at (145.8, 121.0)
- added Q8: BC556, Package_TO_SOT_THT:TO-92_Wide, F.Cu at (155.0, 120.8)
- added Q9: BS170, Package_TO_SOT_THT:TO-92_Wide, F.Cu at (168.2, 131.5)
- added R3: 10k, Resistor_THT:R_Axial_DIN0207_L6.3mm_D2.5mm_P10.16mm_Horizontal, F.Cu at (120.0, 63.6)
- added R6: 4.7k, Resistor_THT:R_Axial_DIN0207_L6.3mm_D2.5mm_P10.16mm_Horizontal, F.Cu at (149.7, 115.0)
- added RV1: 50k, Potentiometer_THT:Potentiometer_Bourns_3296Y_Vertical, F.Cu at (64.5, 64.2)
- added RV3: 50k, Potentiometer_THT:Potentiometer_Bourns_3296Y_Vertical, F.Cu at (78.9, 60.9)
- added U5: DG419LDJ, Package_DIP:DIP-8_W7.62mm_Socket, F.Cu at (131.7, 110.7)
- added U6: LM311, Package_DIP:DIP-8_W7.62mm_Socket, F.Cu at (176.9, 119.4)
- added U7: 4011, Package_DIP:DIP-14_W7.62mm_Socket, F.Cu at (176.7, 69.9)
- C1: value 10u -> 0.1n; footprint Capacitor_THT:CP_Radial_D6.3mm_P2.50mm -> Capacitor_THT:C_Disc_D5.1mm_W3.2mm_P5.00mm
- C11: value 0.1u -> 10n
- C13: value 0.1u -> 0.1n
- C14: value 0.1n -> 0.1u
- C2: value 1u -> 0.1u; footprint Capacitor_THT:C_Rect_L7.2mm_W5.0mm_P5.00mm -> Capacitor_THT:C_Rect_L10.3mm_W4.5mm_P7.50mm_MKS4
- C3: value 0.1u -> 10n; footprint Capacitor_THT:C_Rect_L7.2mm_W2.5mm_P5.00mm -> Capacitor_THT:C_Disc_D5.1mm_W3.2mm_P5.00mm
- C5: value 10n -> 100u; footprint Capacitor_THT:C_Disc_D5.1mm_W3.2mm_P5.00mm -> Capacitor_THT:CP_Radial_D10.0mm_P5.00mm
- C7: value 100u -> 0.1u; footprint Capacitor_THT:CP_Radial_D10.0mm_P5.00mm -> Capacitor_THT:C_Disc_D5.1mm_W3.2mm_P5.00mm
- Q1, Q2: value BC556 -> AS394CH; footprint Package_TO_SOT_THT:TO-92_Wide -> Package_TO_SOT_THT:TO-5-8
- Q3: value BC556 -> AS395H; footprint Package_TO_SOT_THT:TO-92_Wide -> Package_TO_SOT_THT:TO-5-8
- R1: value 9.1k -> 1.2k 1%
- R10, R19: value 22k -> 100k
- R11: value 1k -> 100
- R13, R17, R20: value 22k -> 10k
- R14, R16: value 100k -> 10k
- R15: value 100k -> 22k
- R18, R9: value 10k -> 22k
- R2, R5: value 1k -> 1M
- R21: value 22k -> 1k
- R22: value 10k -> 1k
- R4: value 9.1k -> 470
- R7: value 22k -> 100
- R8: value 4.7k -> 1k
- U1: value TL072 -> 40106; footprint Package_DIP:DIP-8_W7.62mm_Socket -> Package_DIP:DIP-14_W7.62mm_Socket
- U2: value TL072 -> 4013; footprint Package_DIP:DIP-8_W7.62mm_Socket -> Package_DIP:DIP-14_W7.62mm_Socket
- U3: value 4011 -> TL072; footprint Package_DIP:DIP-14_W7.62mm_Socket -> Package_DIP:DIP-8_W7.62mm_Socket
- U4: value 4013 -> TL072; footprint Package_DIP:DIP-14_W7.62mm_Socket -> Package_DIP:DIP-8_W7.62mm_Socket
- moved H3 191.4 mm to (32.3, 83.1)
- moved C7 187.1 mm to (38.0, 33.6), turned to 0 degrees
- moved H2 185.1 mm to (32.3, 75.2)
- moved J1 169.0 mm to (52.6, 78.2), turned to 0 degrees
- moved C12 160.0 mm to (46.2, 28.9)
- moved C6 157.9 mm to (64.4, 34.3), turned to 0 degrees
- moved C5 151.6 mm to (64.4, 22.8), turned to 0 degrees
- moved C9 148.0 mm to (46.2, 19.4), turned to 0 degrees
- moved C8 139.5 mm to (38.0, 38.4), turned to 0 degrees
- moved J14 133.9 mm to (80.3, 82.2)
- moved J13 132.8 mm to (80.3, 78.1)
- moved C10 130.2 mm to (46.2, 24.1), turned to 0 degrees
- moved H4 127.4 mm to (32.3, 91.1)
- moved H1 119.7 mm to (32.3, 67.2)
- moved C14 118.1 mm to (46.2, 33.6), turned to 0 degrees
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Connections:
- C1 pad 1: /SLOW_SW -> Net-(Q1A-C1)
- C1 pad 2: Net-(Q1-C) -> Net-(C1-Pad2)
- C10 pad 1: VCC2 -> GND
- C10 pad 2: GND -> VEE
- C11 pad 1: GND -> VCC
- C11 pad 2: VEE1 -> Net-(U2B-S)
- C12 pad 1: VCC1 -> VCC
- C13 pad 1: VCC1 -> Net-(C13-Pad1)
- C14 pad 1: Net-(U2A--) -> VCC
- C14 pad 2: Net-(C14-Pad2) -> GND
- C2 pad 1: /MED_SW -> Net-(Q2B-C2)
- C2 pad 2: Net-(Q1-C) -> /INT_OUT
- C3 pad 1: /INT_IN -> VCC
- C3 pad 2: Net-(Q1-C) -> Net-(U6-BAL)
- C4 pad 2: Net-(U1B--) -> Net-(C4-Pad2)
- C5 pad 1: VCC1 -> VCC
- C5 pad 2: Net-(U4A-S) -> GND
- C6 pad 1: VCC -> GND
- C6 pad 2: GND -> VEE
- C7 pad 1: GND -> VCC
- C7 pad 2: VEE -> GND
- C8 pad 1: VCC2 -> VCC
- C9 pad 1: GND -> VCC
- C9 pad 2: VEE1 -> GND
- D1 pad 1: /R_FAST -> Net-(D1-K)
- D1 pad 2: /ST_OUT -> Net-(D1-A)
- D2 pad 1: /ST_OUT -> GND
- D2 pad 2: /F_FAST -> Net-(D1-K)
- D5 pad 1: Net-(D5-K) -> VCC
- D5 pad 2: VEE1 -> Net-(D5-A)
- D6 pad 1: Net-(D6-K) -> Net-(D5-A)
- D6 pad 2: /ST_OUT -> GND
- J10 pad 1: /CYCLE_EN -> /R_OUT
- J11 pad 1: /RAMP_OUT -> /F_OUT
- J12 pad 1: /TRIG_IN -> VCC
- J13 pad 1: /RISE_OUT -> VEE
- J14 pad 1: /FALL_OUT -> GND
- J2 pad 1: /R_FAST -> /R_POT_IN
- J3 pad 1: /R_SLOW -> /R_POT_WIPER
- J4 pad 1: /F_FAST -> /F_POT_IN
- J5 pad 1: /F_SLOW -> /F_POT_WIPER
- J6 pad 1: /INT_IN -> /LED
- J7 pad 1: /SLOW_SW -> /CYCLE_EN
- J8 pad 1: /MED_SW -> /RAMP_OUT
- J9 pad 1: /LED -> /TRIG_IN
- Q1 pad 1: Net-(Q1-C) -> Net-(Q1A-C1)
- Q1 pad 2: Net-(D3-A) -> /F_CV
- Q1 pad 3: /INT_IN -> Net-(Q1A-E1)
- Q2 pad 1: /LED -> Net-(Q1A-C1)
- Q2 pad 2: GND -> /R_CV
- Q2 pad 3: Net-(Q2-E) -> Net-(Q2A-E1)
- Q3 pad 1: Net-(Q3-C) -> Net-(Q3A-C1)
- Q3 pad 2: Net-(Q3-B) -> Net-(Q3A-B1)
- Q3 pad 3: VCC2 -> VCC
- Q4 pad 1: Net-(JP2-A) -> Net-(Q3A-C1)
- Q4 pad 2: Net-(D5-K) -> Net-(D1-A)
- Q4 pad 3: Net-(JP3-B) -> Net-(Q1B-C2)
- R1 pad 1: /R_FAST -> Net-(Q1A-C1)
- R1 pad 2: /R_SLOW -> VCC
- R10 pad 1: Net-(C14-Pad2) -> GND
- R10 pad 2: Net-(U2A--) -> Net-(U6-+)
- R11 pad 1: /RAMP_OUT -> Net-(Q9-G)
- R11 pad 2: Net-(C14-Pad2) -> Net-(C4-Pad1)
- R12 pad 1: Net-(Q3-C) -> Net-(U6-+)
- R12 pad 2: VEE1 -> /CMP_OUT
- R13 pad 1: Net-(C14-Pad2) -> Net-(C4-Pad1)
- R13 pad 2: Net-(JP1-B) -> VEE
- R14 pad 1: Net-(Q3-B) -> /CMP_OUT
- R14 pad 2: Net-(JP6-B) -> VCC
- R15 pad 1: Net-(U2B-+) -> Net-(C4-Pad2)
- R15 pad 2: GND -> /RESET
- R16 pad 1: Net-(D5-K) -> Net-(Q10-D)
- R16 pad 2: Net-(C4-Pad1) -> VCC
- R17 pad 1: Net-(U2B-+) -> Net-(D5-A)
- R17 pad 2: Net-(D6-K) -> /TRIG_IN
- R18 pad 1: Net-(C4-Pad1) -> /CLK
- R18 pad 2: VEE1 -> Net-(C13-Pad1)
- R19 pad 1: /ST_OUT -> /TRIG_IN
- R19 pad 2: /CLK -> GND
- R2 pad 2: /R_SLOW -> Net-(Q1A-E1)
- R20 pad 1: Net-(U4A-S) -> Net-(U2B-S)
- R21 pad 1: Net-(U1B--) -> Net-(R21-Pad1)
- R21 pad 2: /CYCLE_EN -> /R_OUT
- R22 pad 1: Net-(D7-K) -> Net-(R22-Pad1)
- R22 pad 2: /TRIG_IN -> /F_OUT
- R4 pad 1: /F_FAST -> Net-(C1-Pad2)
- R4 pad 2: /F_SLOW -> Net-(R4-Pad2)
- R5 pad 2: /F_SLOW -> Net-(Q2A-E1)
- R7 pad 1: Net-(U2A--) -> Net-(Q6-G)
- R7 pad 2: Net-(Q1-C) -> /Q
- R8 pad 1: Net-(C14-Pad2) -> /RAMP_OUT
- R8 pad 2: Net-(Q2-E) -> /INT_OUT
- R9 pad 1: Net-(Q3-C) -> /INT_OUT
- R9 pad 2: Net-(D3-A) -> Net-(Q9-D)
- U1 pad 1: Net-(Q1-C) -> /CMP_OUT
- U1 pad 2: /INT_IN -> Net-(U1-Pad2)
- U1 pad 3: GND -> Net-(U1-Pad2)
- U1 pad 4: VEE1 -> /CLK
- U1 pad 5: Net-(D7-K) -> GND
- U1 pad 6: Net-(U1B--) -> unconnected-(U1-Pad6)
- U1 pad 7: Net-(U1B--) -> GND
- U1 pad 8: VCC2 -> Net-(C4-Pad2)
- U2 pad 1: Net-(C14-Pad2) -> unconnected-(U2A-Q-Pad1)
- U2 pad 2: Net-(U2A--) -> unconnected-(U2A-~{Q}-Pad2)
- U2 pad 4: VEE1 -> GND
- U2 pad 5: Net-(U2B-+) -> GND
- U2 pad 6: Net-(JP1-B) -> GND
- U2 pad 7: /ST_OUT -> GND
- U2 pad 8: VCC2 -> Net-(U2B-S)
- U3 pad 1: Net-(JP7-B) -> /F_CV
- U3 pad 2: /CLK -> /F_CV
- U3 pad 3: Net-(JP10-A) -> /F_POT_WIPER
- U3 pad 4: Net-(R23-Pad1) -> VEE
- U3 pad 5: Net-(JP5-A) -> /R_POT_WIPER
- U3 pad 6: Net-(JP5-A) -> /R_CV
- U3 pad 7: GND -> /R_CV
- U3 pad 8: Net-(JP10-B) -> VCC
- U4 pad 1: Net-(JP6-A) -> Net-(C1-Pad2)
- U4 pad 2: Net-(JP7-A) -> Net-(Q1A-C1)
- U4 pad 3: /CLK -> GND
- U4 pad 4: Net-(JP4-B) -> VEE
- U4 pad 5: VCC1 -> GND
- U4 pad 6: Net-(U4A-S) -> Net-(Q2B-C2)
- U4 pad 7: GND -> /INT_OUT
- U4 pad 8: GND -> VCC
Routing:
- net GND: track 533.3 -> 0.00 mm
- net VCC2: track 77.0 -> 0.00 mm
- net Net-(JP6-A): track 72.2 -> 0.00 mm
- net VCC1: track 72.1 -> 0.00 mm
- net VEE1: track 53.8 -> 0.00 mm
- net VEE: track 52.1 -> 0.00 mm
- net Net-(C14-Pad2): track 50.8 -> 0.00 mm
- net /CLK: track 46.8 -> 0.00 mm
- net VCC: track 43.7 -> 0.00 mm
- net Net-(JP1-B): track 35.9 -> 0.00 mm
- net Net-(Q1-C): track 26.9 -> 0.00 mm
- net Net-(JP10-A): track 23.6 -> 0.00 mm
- net Net-(JP4-B): track 22.5 -> 0.00 mm
- net Net-(JP1-A): track 20.3 -> 0.00 mm
- net Net-(JP10-B): track 18.5 -> 0.00 mm
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Other:
- board size 75 x 100 mm -> 80 x 110 mm

Commit message: delete jumpers library
Parts:
- removed RV3: 50k, Potentiometer_THT:Potentiometer_Bourns_3296Y_Vertical
- added C16: 0.1u, Capacitor_THT:C_Disc_D5.1mm_W3.2mm_P5.00mm, F.Cu at (96.0, 59.0)
- added C17: 0.1u, Capacitor_THT:C_Disc_D5.1mm_W3.2mm_P5.00mm, F.Cu at (96.0, 74.0)
- added C18: 0.1u, Capacitor_THT:C_Disc_D5.1mm_W3.2mm_P5.00mm, F.Cu at (96.0, 81.5)
- added C19: 0.1u, Capacitor_THT:C_Disc_D5.1mm_W3.2mm_P5.00mm, F.Cu at (96.0, 96.5)
- added J10: Conn_01x01, Connector_Pin:Pin_D1.0mm_L10.0mm, F.Cu at (62.2, 65.0)
- added J6: Conn_01x01, Connector_Pin:Pin_D1.0mm_L10.0mm, F.Cu at (32.1, 75.1)
- added J7: Conn_01x01, Connector_Pin:Pin_D1.0mm_L10.0mm, F.Cu at (31.1, 49.5)
- added J8: Conn_01x01, Connector_Pin:Pin_D1.0mm_L10.0mm, F.Cu at (32.1, 70.1)
- added J9: Conn_01x01, Connector_Pin:Pin_D1.0mm_L10.0mm, F.Cu at (31.1, 44.5)
- added R10: 22k, Resistor_THT:R_Axial_DIN0207_L6.3mm_D2.5mm_P10.16mm_Horizontal, F.Cu at (55.2, 51.6)
- added R11: 22k, Resistor_THT:R_Axial_DIN0207_L6.3mm_D2.5mm_P10.16mm_Horizontal, F.Cu at (51.8, 68.5)
- added R12: 22k, Resistor_THT:R_Axial_DIN0207_L6.3mm_D2.5mm_P10.16mm_Horizontal, F.Cu at (51.0, 45.0)
- added R3: 22k, Resistor_THT:R_Axial_DIN0207_L6.3mm_D2.5mm_P10.16mm_Horizontal, F.Cu at (49.0, 63.0)
- added R4: 22k, Resistor_THT:R_Axial_DIN0207_L6.3mm_D2.5mm_P10.16mm_Horizontal, F.Cu at (49.0, 66.5)
- added R5: 22k, Resistor_THT:R_Axial_DIN0207_L6.3mm_D2.5mm_P10.16mm_Horizontal, F.Cu at (49.0, 88.5)
- added R6: 22k, Resistor_THT:R_Axial_DIN0207_L6.3mm_D2.5mm_P10.16mm_Horizontal, F.Cu at (62.2, 51.6)
- added R7: 22k, Resistor_THT:R_Axial_DIN0207_L6.3mm_D2.5mm_P10.16mm_Horizontal, F.Cu at (55.2, 85.1)
- added R8: 22k, Resistor_THT:R_Axial_DIN0207_L6.3mm_D2.5mm_P10.16mm_Horizontal, F.Cu at (58.7, 61.8)
- added R9: 22k, Resistor_THT:R_Axial_DIN0207_L6.3mm_D2.5mm_P10.16mm_Horizontal, F.Cu at (58.7, 74.9)
- added RV5: 50k, Potentiometer_THT:Potentiometer_Bourns_3296Y_Vertical, F.Cu at (-65.0, 46.6)
- added U4: TL074, Package_DIP:DIP-14_W7.62mm_Socket, F.Cu at (47.7, 59.6)
- U3: value TL072 -> TL074; footprint Package_DIP:DIP-8_W7.62mm_Socket -> Package_DIP:DIP-14_W7.62mm_Socket
- moved Q7 156.2 mm to (166.7, -33.7)
- moved R18 156.2 mm to (170.7, -39.8)
- moved Q8 156.2 mm to (175.9, -34.0)
- moved J11 152.4 mm to (172.7, -30.3)
- moved R25 120.8 mm to (75.8, 81.5), turned to 0 degrees
- moved C11 118.6 mm to (-57.5, -28.8)
- moved C3 118.6 mm to (-39.2, -34.9)
- moved C4 118.6 mm to (-39.2, -23.3)
- moved H1 118.6 mm to (-71.4, 9.58)
- moved H2 118.6 mm to (-71.4, 17.5)
- moved H3 118.6 mm to (-71.4, 25.5)
- moved H4 118.6 mm to (-71.4, 33.4)
- moved J17 118.6 mm to (-23.4, 16.4)
- moved J18 118.6 mm to (-23.4, 20.4)
- moved J19 118.6 mm to (-23.4, 24.5)
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- renumbered C12 to C11, C14 to C12, C15 to C13, C16 to C14, C17 to C15, C11 to C20, C13 to C21, C5 to C3, C6 to C4, C7 to C5, C3 to C6, C8 to C7, C4 to C8, J6 to J11, J7 to J12, J8 to J13, J9 to J14, J10 to J15, J11 to J16, J12 to J17, J13 to J18, J14 to J19, R1 to R13, R2 to R14, R3 to R15, R4 to R16, R5 to R17, R6 to R18, R7 to R19, R8 to R20, R9 to R21, R10 to R22, R11 to R23, R12 to R24, R13 to R25, R14 to R26, R15 to R27, R16 to R28, R17 to R29, R18 to R30, R19 to R31, R20 to R32, R21 to R33, R22 to R34, RV1 to RV2, U4 to U5, U5 to U6, U6 to U7, U7 to U8
Connections:
- C20 pad 2: Net-(U2B-S) -> Net-(U2A-S)
- C21 pad 1: Net-(C13-Pad1) -> Net-(C21-Pad1)
- C8 pad 2: Net-(C4-Pad2) -> Net-(C8-Pad2)
- J3 pad 1: /R_POT_WIPER -> /R_WIPER
- J5 pad 1: /F_POT_WIPER -> /F_WIPER
- R27 pad 1: Net-(C4-Pad2) -> Net-(C8-Pad2)
- R30 pad 2: Net-(C13-Pad1) -> Net-(C21-Pad1)
- R32 pad 1: Net-(U2B-S) -> Net-(U2A-S)
- U1 pad 1: /CMP_OUT -> Net-(Q10-D)
- U1 pad 10: unconnected-(U1-Pad10) -> Net-(U1-Pad10)
- U1 pad 11: GND -> /CMP_OUT
- U1 pad 12: Net-(U1-Pad12) -> unconnected-(U1-Pad12)
- U1 pad 13: Net-(C13-Pad1) -> GND
- U1 pad 2: Net-(U1-Pad2) -> Net-(C8-Pad2)
- U1 pad 3: Net-(U1-Pad2) -> Net-(C21-Pad1)
- U1 pad 4: /CLK -> Net-(U1-Pad4)
- U1 pad 8: Net-(C4-Pad2) -> /CLK
- U1 pad 9: Net-(Q10-D) -> Net-(U1-Pad10)
- U2 pad 1: unconnected-(U2A-Q-Pad1) -> /Q
- U2 pad 10: /RESET -> GND
- U2 pad 11: /CLK -> GND
- U2 pad 12: /~{Q} -> unconnected-(U2B-~{Q}-Pad12)
- U2 pad 13: /Q -> unconnected-(U2B-Q-Pad13)
- U2 pad 2: unconnected-(U2A-~{Q}-Pad2) -> /~{Q}
- U2 pad 3: GND -> /CLK
- U2 pad 4: GND -> /RESET
- U2 pad 5: GND -> VCC
- U2 pad 6: GND -> Net-(U2A-S)
- U2 pad 8: Net-(U2B-S) -> GND
- U2 pad 9: VCC -> GND
- U3 pad 1: /F_CV -> Net-(R7-Pad1)
- U3 pad 2: /F_CV -> Net-(U3A--)
- U3 pad 3: /F_POT_WIPER -> GND
- U3 pad 4: VEE -> VCC
- U3 pad 5: /R_POT_WIPER -> GND
- U3 pad 6: /R_CV -> Net-(U3B--)
- U3 pad 8: VCC -> /R_CV_BUF
- U8 pad 8: Net-(U1-Pad12) -> Net-(U1-Pad4)
- U8 pad 9: Net-(U1-Pad12) -> Net-(U1-Pad4)
Other:
- board size 80 x 110 mm -> 90 x 110 mm

Commit message: small tweaks
Parts:
- removed C19: 0.1u, Capacitor_THT:C_Disc_D5.1mm_W3.2mm_P5.00mm
- removed C20: 10n, Capacitor_THT:C_Disc_D5.1mm_W3.2mm_P5.00mm
- removed C21: 0.1n, Capacitor_THT:C_Disc_D5.1mm_W3.2mm_P5.00mm
- removed J1: Conn_02x05_Odd_Even, Connector_IDC:IDC-Header_2x05_P2.54mm_Vertical
- removed J2: Conn_01x01, Connector_Pin:Pin_D1.0mm_L10.0mm
- removed Q10, Q9: BS170, Package_TO_SOT_THT:TO-92_Wide
- removed Q8: BC556, Package_TO_SOT_THT:TO-92_Wide
- removed RV2: 50k, Potentiometer_THT:Potentiometer_Bourns_3296Y_Vertical
- removed U7: LM311, Package_DIP:DIP-8_W7.62mm_Socket
- removed U8: 4011, Package_DIP:DIP-14_W7.62mm_Socket
- added D7: 1N4148, Diode_THT:D_DO-35_SOD27_P7.62mm_Horizontal, F.Cu at (148.0, 106.2)
- added D8: 1N4148, Diode_THT:D_DO-35_SOD27_P7.62mm_Horizontal, F.Cu at (148.0, 117.0)
- added J20: Conn_01x01, Connector_Pin:Pin_D1.0mm_L10.0mm, F.Cu at (153.0, 141.5)
- added J21: Conn_01x01, Connector_Pin:Pin_D1.0mm_L10.0mm, F.Cu at (158.0, 141.5)
- added R35: 1k, Resistor_THT:R_Axial_DIN0207_L6.3mm_D2.5mm_P10.16mm_Horizontal, F.Cu at (183.0, 111.1)
- added RV6: 50k, Potentiometer_THT:Potentiometer_Bourns_3296Y_Vertical, F.Cu at (146.0, 135.3)
- C15, C17: value 0.1u -> 0.1n
- C16: value 0.1u -> 10n
- C18: value 0.1u -> 1n
- C2: value 0.1u -> 0.1n; footprint Capacitor_THT:C_Rect_L10.3mm_W4.5mm_P7.50mm_MKS4 -> Capacitor_THT:C_Disc_D5.1mm_W3.2mm_P5.00mm
- C3: value 100u -> 47n; footprint Capacitor_THT:CP_Radial_D10.0mm_P5.00mm -> Capacitor_THT:C_Rect_L13.0mm_W5.0mm_P10.00mm_FKS3_FKP3_MKS4
- C5: value 0.1u -> 100u; footprint Capacitor_THT:C_Disc_D5.1mm_W3.2mm_P5.00mm -> Capacitor_THT:CP_Radial_D10.0mm_P5.00mm
- C6: value 10n -> 0.1u
- C8: value 0.1n -> 0.1u
- J3: value Conn_01x01 -> Conn_02x05_Odd_Even; footprint Connector_Pin:Pin_D1.0mm_L10.0mm -> Connector_IDC:IDC-Header_2x05_P2.54mm_Vertical
- Q1: value AS394CH -> AS395H
- Q3: value AS395H -> BS170; footprint Package_TO_SOT_THT:TO-5-8 -> Package_TO_SOT_THT:TO-92_Wide
- Q7: value BC546 -> BS170
- R10, R27, R3, R30, R4, R5, R6, R7, R8, R9: value 22k -> 10k
- R11, R12: value 22k -> 2.2M
- R13: value 1.2k 1% -> 2.2k 1%
- R14: value 1M -> 2.2k 1%
- R15: value 10k -> 820
- R16: value 470 -> 820
- R17: value 1M -> 1k
- R18: value 4.7k -> 100
- R19: value 100 -> 4.7k
- R20: value 1k -> 10k
- R21: value 22k -> 68k
- R22: value 100k -> 100
- R23: value 100 -> 10k
- R25: value 10k -> 33k
- R28: value 10k -> 22k
- R29: value 10k -> 47k
- R31: value 100k -> 10k
- R33: value 1k -> 100k
- U1: value 40106 -> TL074
- U2: value 4013 -> TL074
- U4: value TL074 -> 4013
- U5: value TL072 -> 4011; footprint Package_DIP:DIP-8_W7.62mm_Socket -> Package_DIP:DIP-14_W7.62mm_Socket
- U6: value DG419LDJ -> 40106; footprint Package_DIP:DIP-8_W7.62mm_Socket -> Package_DIP:DIP-14_W7.62mm_Socket
- moved H3 284.8 mm to (188.5, 142.0)
- moved C11 269.4 mm to (175.5, 106.5), turned to -90 degrees
- moved C4 262.1 mm to (176.5, 125.6), turned to -90 degrees
- moved H1 261.9 mm to (188.5, 42.0)
- moved C3 236.1 mm to (176.5, 61.0), turned to 90 degrees
- moved J17 226.7 mm to (188.5, 97.0)
- moved J18 223.6 mm to (188.5, 92.0)
- moved H4 223.1 mm to (123.5, 142.0)
- moved RV5 219.2 mm to (135.5, 135.3), turned to 180 degrees
- moved J19 207.5 mm to (148.0, 141.5)
- moved J4 201.8 mm to (133.0, 141.5)
- moved H2 196.4 mm to (123.5, 42.0)
- moved J3 164.4 mm to (188.5, 130.6), turned to 180 degrees
- moved Q7 155.9 mm to (137.7, 119.5), turned to -90 degrees
- moved C10 141.9 mm to (175.5, 85.0), turned to -90 degrees
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Connections:
- C1 pad 1: Net-(Q1A-C1) -> Net-(Q2A-C1)
- C10 pad 1: GND -> VCC
- C10 pad 2: VEE -> GND
- C12 pad 1: VCC -> GND
- C12 pad 2: GND -> VEE
- C13 pad 1: GND -> VCC
- C13 pad 2: VEE -> GND
- C14 pad 1: VCC -> GND
- C14 pad 2: GND -> VEE
- C15 pad 1: GND -> Net-(C15-Pad1)
- C15 pad 2: VEE -> Net-(C15-Pad2)
- C16 pad 2: GND -> Net-(U4A-S)
- C17 pad 1: GND -> Net-(C17-Pad1)
- C17 pad 2: VEE -> GND
- C18 pad 1: VCC -> Net-(C18-Pad1)
- C18 pad 2: GND -> Net-(Q7-D)
- C2 pad 1: Net-(Q2B-C2) -> Net-(Q1B-C2)
- C2 pad 2: /INT_OUT -> Net-(C2-Pad2)
- C3 pad 1: VCC -> Net-(Q1A-C1)
- C3 pad 2: GND -> /INT_OUT
- C4 pad 1: GND -> VCC
- C4 pad 2: VEE -> GND
- C5 pad 1: VCC -> GND
- C5 pad 2: GND -> VEE
- C6 pad 2: Net-(U7-BAL) -> GND
- C8 pad 1: Net-(C8-Pad1) -> VCC
- C8 pad 2: Net-(C8-Pad2) -> GND
- C9 pad 1: VCC -> GND
- C9 pad 2: GND -> VEE
- D1 pad 1: Net-(D1-K) -> /CMP_OUT
- D2 pad 1: GND -> Net-(D2-K)
- D2 pad 2: Net-(D1-K) -> /CMP_OUT
- D4 pad 1: /RESET -> Net-(D4-K)
- D4 pad 2: /CYCLE_EN -> /CMP_OUT
- D5 pad 1: VCC -> /CLK
- D5 pad 2: Net-(D5-A) -> GND
- D6 pad 1: Net-(D5-A) -> /RESET
- D6 pad 2: GND -> /CYCLE_EN
- J10 pad 1: /F_CV_SUM_IN -> /R_CV_BUF
- J11 pad 1: /LED -> /F_CV_BUF
- J12 pad 1: /CYCLE_EN -> /F_CV_SUM_IN
- J13 pad 1: /RAMP_OUT -> /LED
- J14 pad 1: /TRIG_IN -> /CYCLE_EN
- J15 pad 1: /R_OUT -> /RAMP_OUT
- J16 pad 1: /F_OUT -> /TRIG_IN
- J17 pad 1: VCC -> /R_OUT
- J18 pad 1: VEE -> /F_OUT
- J19 pad 1: GND -> VCC
- J3 pad 1: /R_WIPER -> VEE
- J4 pad 1: /F_POT_IN -> /R_POT_IN
- J5 pad 1: /F_WIPER -> /R_WIPER
- J6 pad 1: /R_CV_WIPER -> /F_POT_IN
- J7 pad 1: /F_CV_WIPER -> /F_WIPER
- J8 pad 1: /R_CV_BUF -> /R_CV_WIPER
- J9 pad 1: /F_CV_BUF -> /F_CV_WIPER
- Q1 pad 2: /F_CV -> GND
- Q1 pad 6: GND -> /F_CV
- Q2 pad 1: Net-(Q1A-C1) -> Net-(Q2A-C1)
- Q2 pad 7: Net-(Q2B-C2) -> Net-(Q1A-C1)
- Q3 pad 1: Net-(Q3A-C1) -> /INT_OUT
- Q3 pad 2: Net-(Q3A-B1) -> Net-(Q3-G)
- Q3 pad 3: VCC -> Net-(Q1A-C1)
- Q4 pad 1: Net-(Q3A-C1) -> VCC
- Q4 pad 2: Net-(D1-A) -> /INT_OUT
- Q4 pad 3: Net-(Q1B-C2) -> Net-(Q4-E)
- Q5 pad 1: Net-(Q2B-C2) -> /LED
- Q5 pad 2: Net-(Q3A-C1) -> GND
- Q5 pad 3: Net-(Q3A-B1) -> Net-(Q5-E)
- Q6 pad 1: /INT_OUT -> Net-(Q6-D)
- Q6 pad 3: Net-(Q2B-C2) -> VEE
- Q7 pad 1: VCC -> Net-(Q7-D)
- Q7 pad 2: /INT_OUT -> Net-(D7-A)
- Q7 pad 3: Net-(Q7-E) -> GND
- R10 pad 1: Net-(U4B--) -> /R_CV
- R10 pad 2: Net-(R10-Pad2) -> Net-(U1A--)
- R11 pad 1: /R_CV -> VEE
- R11 pad 2: Net-(U3B--) -> Net-(D1-A)
- R12 pad 1: /F_CV -> VCC
- R12 pad 2: Net-(U4B--) -> Net-(D2-K)
- R13 pad 1: Net-(Q1A-C1) -> Net-(D1-A)
- R13 pad 2: VCC -> Net-(Q1B-C2)
- R14 pad 1: GND -> Net-(Q2A-C1)
- R14 pad 2: Net-(Q1A-E1) -> Net-(D2-K)
- R15 pad 1: Net-(D1-A) -> Net-(Q1A-E1)
- R15 pad 2: VCC -> Net-(C2-Pad2)
- R16 pad 2: Net-(R16-Pad2) -> Net-(Q2A-E1)
- R17 pad 1: GND -> /RAMP_OUT
- R17 pad 2: Net-(Q2A-E1) -> /INT_OUT
- R18 pad 1: Net-(Q7-E) -> Net-(Q3-G)
- R18 pad 2: Net-(Q8-E) -> /Q
- R19 pad 1: Net-(Q6-G) -> Net-(Q4-E)
- R19 pad 2: /Q -> Net-(Q5-E)
- R20 pad 1: /RAMP_OUT -> /INT_OUT
- R20 pad 2: /INT_OUT -> Net-(Q6-D)
- R21 pad 1: /INT_OUT -> GND
- R21 pad 2: Net-(Q9-D) -> Net-(U3A-+)
- R22 pad 1: GND -> Net-(Q6-G)
- R22 pad 2: Net-(U7-+) -> Net-(C15-Pad1)
- R23 pad 1: Net-(Q9-G) -> Net-(D4-K)
- R23 pad 2: Net-(C8-Pad1) -> Net-(U3A-+)
- R24 pad 1: Net-(U7-+) -> Net-(C15-Pad1)
- R24 pad 2: /CMP_OUT -> VEE
- R25 pad 1: Net-(C8-Pad1) -> Net-(C15-Pad2)
- R25 pad 2: VEE -> /RESET
- R26 pad 2: VCC -> /CLK
- R27 pad 1: Net-(C8-Pad2) -> Net-(C18-Pad1)
- R27 pad 2: /RESET -> Net-(R27-Pad2)
- R28 pad 1: Net-(Q10-D) -> /CLK
- R28 pad 2: VCC -> Net-(C17-Pad1)
- R29 pad 1: Net-(D5-A) -> Net-(C18-Pad1)
- R29 pad 2: /TRIG_IN -> VCC
- R3 pad 1: Net-(U4A--) -> Net-(U2B--)
- R3 pad 2: Net-(U4D--) -> Net-(U2C--)
- R30 pad 1: /CLK -> Net-(U4A-S)
- R30 pad 2: Net-(C21-Pad1) -> GND
- R31 pad 1: /TRIG_IN -> Net-(Q7-D)
- R31 pad 2: GND -> VCC
- R32 pad 1: Net-(U2A-S) -> Net-(D7-A)
- R32 pad 2: GND -> /TRIG_IN
- R33 pad 1: Net-(R33-Pad1) -> /TRIG_IN
- R33 pad 2: /R_OUT -> GND
- R34 pad 2: /F_OUT -> /R_OUT
- R4 pad 1: Net-(U3A--) -> Net-(U1B--)
- R4 pad 2: /R_CV_BUF -> Net-(U1C--)
- R5 pad 1: Net-(U3A--) -> Net-(U2B--)
- R5 pad 2: Net-(U3D--) -> /R_CV_BUF
- R6 pad 1: Net-(U4A--) -> Net-(U1B--)
- R7 pad 1: Net-(R7-Pad1) -> /F_CV
- R7 pad 2: Net-(U3A--) -> Net-(U1B--)
- R8 pad 1: Net-(R10-Pad2) -> Net-(R8-Pad1)
- R8 pad 2: Net-(U4A--) -> Net-(U2B--)
- R9 pad 1: Net-(U3B--) -> Net-(U1A--)
- R9 pad 2: Net-(R7-Pad1) -> Net-(R8-Pad1)
- RV5 pad 3: /F_POT_IN -> /R_POT_IN
- U1 pad 1: Net-(Q10-D) -> /R_CV
- U1 pad 10: Net-(U1-Pad10) -> /F_WIPER
- U1 pad 11: /CMP_OUT -> VEE
- U1 pad 12: unconnected-(U1-Pad12) -> /F_CV_WIPER
- U1 pad 13: GND -> /F_CV_BUF
- U1 pad 14: VCC -> /F_CV_BUF
- U1 pad 2: Net-(C8-Pad2) -> Net-(U1A--)
- U1 pad 3: Net-(C21-Pad1) -> GND
- U1 pad 4: Net-(U1-Pad4) -> VCC
- U1 pad 6: unconnected-(U1-Pad6) -> Net-(U1B--)
- U1 pad 7: GND -> /F_CV
- U1 pad 8: /CLK -> Net-(U1C--)
- U1 pad 9: Net-(U1-Pad10) -> Net-(U1C--)
- U2 pad 1: /Q -> Net-(U2A--)
- U2 pad 10: GND -> /R_WIPER
- U2 pad 11: GND -> VEE
- U2 pad 12: unconnected-(U2B-~{Q}-Pad12) -> /R_CV_WIPER
- U2 pad 13: unconnected-(U2B-Q-Pad13) -> /R_CV_BUF
- U2 pad 14: VCC -> /R_CV_BUF
- U2 pad 2: /~{Q} -> Net-(U2A--)
- U2 pad 3: /CLK -> GND
- U2 pad 4: /RESET -> VCC
- U2 pad 5: VCC -> GND
- U2 pad 6: Net-(U2A-S) -> Net-(U2B--)
- U2 pad 7: GND -> Net-(R8-Pad1)
- U2 pad 8: GND -> Net-(U2C--)
- U2 pad 9: GND -> Net-(U2C--)
- U3 pad 1: Net-(R7-Pad1) -> /CMP_OUT
- U3 pad 10: /R_CV_WIPER -> GND
- U3 pad 12: /R_WIPER -> GND
- U3 pad 13: Net-(U3D--) -> Net-(Q2A-C1)
- U3 pad 14: Net-(U3D--) -> Net-(C1-Pad2)
- U3 pad 2: Net-(U3A--) -> Net-(Q6-D)
- U3 pad 3: GND -> Net-(U3A-+)
- U3 pad 6: Net-(U3B--) -> Net-(Q1A-C1)
- U3 pad 7: /R_CV -> /INT_OUT
- U3 pad 8: /R_CV_BUF -> Net-(C2-Pad2)
- U3 pad 9: /R_CV_BUF -> Net-(Q1B-C2)
- U4 pad 1: Net-(R10-Pad2) -> /Q
- U4 pad 10: /F_CV_WIPER -> GND
- U4 pad 11: VEE -> GND
- U4 pad 12: /F_WIPER -> unconnected-(U4B-~{Q}-Pad12)
- U4 pad 13: Net-(U4D--) -> unconnected-(U4B-Q-Pad13)
- U4 pad 14: Net-(U4D--) -> VCC
- U4 pad 2: Net-(U4A--) -> /~{Q}
- U4 pad 3: GND -> /CLK
- U4 pad 4: VCC -> /RESET
- U4 pad 5: GND -> VCC
- U4 pad 6: Net-(U4B--) -> Net-(U4A-S)
- U4 pad 7: /F_CV -> GND
- U4 pad 8: /F_CV_BUF -> GND
- U4 pad 9: /F_CV_BUF -> GND
- U5 pad 1: Net-(C1-Pad2) -> /~{Q}
- U5 pad 2: Net-(Q1A-C1) -> Net-(U5-Pad2)
- U5 pad 3: GND -> Net-(U5-Pad3)
- U5 pad 4: VEE -> Net-(U5-Pad2)
- U5 pad 5: GND -> Net-(U5-Pad5)
- U5 pad 6: Net-(Q2B-C2) -> Net-(U5-Pad5)
- U5 pad 7: /INT_OUT -> GND
- U5 pad 8: VCC -> Net-(U5-Pad3)
- U6 pad 1: Net-(R16-Pad2) -> GND
- U6 pad 2: Net-(Q1A-E1) -> unconnected-(U6-Pad2)
- U6 pad 4: VCC -> unconnected-(U6-Pad4)
- U6 pad 5: VCC -> GND
- U6 pad 6: /CLK -> unconnected-(U6-Pad6)
- U6 pad 7: VEE -> GND
- U6 pad 8: Net-(Q2A-E1) -> Net-(U5-Pad5)
Routing:
- net VCC: track 0.00 -> 311.7 mm, vias 0 -> 1
- net VEE: track 0.00 -> 267.8 mm, vias 0 -> 4
- net Net-(Q1A-C1): track 0.00 -> 52.9 mm
- net /CLK: track 0.00 -> 47.9 mm
- net Net-(U2B--): track 0.00 -> 45.6 mm
- net Net-(Q6-D): track 0.00 -> 45.2 mm, vias 0 -> 2
- net /INT_OUT: track 0.00 -> 43.4 mm
- net Net-(C15-Pad2): track 0.00 -> 39.8 mm, vias 0 -> 1
- net /~{Q}: track 0.00 -> 38.1 mm
- net Net-(U5-Pad5): track 0.00 -> 37.4 mm
- net /CMP_OUT: track 0.00 -> 36.6 mm
- net Net-(Q2A-C1): track 0.00 -> 27.7 mm
- net /CYCLE_EN: track 0.00 -> 27.4 mm, vias 0 -> 1
- net Net-(C17-Pad1): track 0.00 -> 27.0 mm
- net Net-(U1B--): track 0.00 -> 26.9 mm
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- added copper zone on B.Cu, net GND
Other:
- board size 90 x 110 mm -> 75 x 110 mm
- board text added: "Fall range"
- board text added: "Rise range"

Commit message: threshold pot
Parts:
- removed the R21 at (188.6, 65.5)
- added RV7: 50k, Potentiometer_THT:Potentiometer_Bourns_3296Y_Vertical, F.Cu at (177.7, 72.5)
- moved R23 7.22 mm to (176.9, 68.0), turned to 0 degrees
- moved R20 5.00 mm to (185.6, 65.0)
- moved R17 2.12 mm to (184.0, 81.1)
- moved C11 2.00 mm to (175.5, 108.5)
- moved Q3 1.96 mm to (181.7, 55.5)
- moved R27 1.50 mm to (156.0, 106.4)
- moved Q5 1.00 mm to (189.3, 77.5)
- moved Q6 1.00 mm to (154.8, 88.5)
- moved C3 0.50 mm to (176.5, 60.5)
- renumbered R22 to R21, R24 to R22, R25 to R24, R26 to R25, R27 to R26, R28 to R27, R29 to R28, R30 to R29, R31 to R30, R32 to R31, R33 to R32, R34 to R33, R35 to R34
Connections:
- R23 pad 1: Net-(D4-K) -> Net-(R23-Pad1)
- R23 pad 2: Net-(U3A-+) -> GND
Routing:
- net Net-(U3A-+): track 7.84 -> 18.3 mm
- net Net-(Q6-D): track 45.2 -> 39.8 mm, vias 2 -> 1
- net Net-(R23-Pad1): track 0.00 -> 4.79 mm
- net /~{Q}: track 38.1 -> 42.0 mm
- net /INT_OUT: track 43.4 -> 40.0 mm
- net Net-(Q3-G): track 25.3 -> 28.6 mm
- net /CLK: track 47.9 -> 50.9 mm
- net Net-(D4-K): track 3.86 -> 6.75 mm
- net /Q: track 7.45 -> 5.44 mm
- net Net-(Q1A-C1): track 52.9 -> 51.3 mm
- net VEE: track 267.8 -> 268.8 mm
- net Net-(Q6-G): track 7.15 -> 6.15 mm
- net Net-(Q5-E): track 12.2 -> 11.3 mm
- net Net-(R34-Pad1): track 12.6 -> 13.5 mm
- net Net-(C17-Pad1): track 27.0 -> 27.7 mm
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
Commit message: prettier solder pins arrangement
Parts:
- moved J12 38.4 mm to (121.5, 52.5)
- moved R4 13.9 mm to (139.1, 49.0)
- moved C6 11.8 mm to (137.5, 59.0), turned to 90 degrees
- moved R7 7.91 mm to (142.0, 48.4), turned to -90 degrees
- moved R6 1.94 mm to (141.6, 45.0), turned to 180 degrees
Routing:
- net Net-(U1C--): track 22.7 -> 7.25 mm
- net VCC: track 312.2 -> 302.1 mm
- net /F_CV_SUM_IN: track 9.40 -> 13.1 mm
- net Net-(U1B--): track 26.9 -> 29.0 mm
- net /F_CV: track 23.1 -> 21.1 mm
